Commit message: Add xacro: prefix as required by xacro.py Hydro changes

File: turtlebot_arm_description/urdf/arm.urdf.xacro (robot description, xacro)
@@ -1,4 +1,4 @@
 <?xml version="1.0"?>
-<robot name="turtlebot_arm"
+<robot name="turtlebot_arm" xmlns:xacro="http://ros.org/wiki/xacro"
     xmlns:sensor="http://playerstage.sourceforge.net/gazebo/xmlschema/#sensor"
     xmlns:controller="http://playerstage.sourceforge.net/gazebo/xmlschema/#controller"
@@ -6,5 +6,5 @@
     <!-- Included URDF Files -->
     <!--<include filename="$(find turtlebot_description)/urdf/turtlebot.urdf.xacro" />-->
-    <include filename="$(find turtlebot_arm_description)/urdf/arm.xacro" />
+    <xacro:include filename="$(find turtlebot_arm_description)/urdf/arm.xacro" />
     <!-- For now I have removed the turtlebot since this all moved around..
     <turtlebot />-->

File: turtlebot_arm_description/urdf/arm.xacro (robot description, xacro)
@@ -1,5 +1,5 @@
 <?xml version="1.0"?>
-<robot>
-  <include filename="$(find turtlebot_arm_description)/urdf/arm_hardware.xacro" />
+<robot xmlns:xacro="http://ros.org/wiki/xacro">
+  <xacro:include filename="$(find turtlebot_arm_description)/urdf/arm_hardware.xacro"/>
   <material name="white">
     <color rgba="0.87 0.90 0.87 1.0"/>
@@ -11,5 +11,5 @@
     <color rgba="0.22 0.32 0.14 1.0"/>
   </material>
-  <macro name="turtlebot_arm" params="parent color gripper_color *origin">
+  <xacro:macro name="turtlebot_arm" params="parent color gripper_color *origin">
     <link name="arm_base_link" />
     <joint name="arm_base_joint" type="fixed">
@@ -128,4 +128,4 @@
       <origin xyz="0 0 0" rpy="0 0 ${M_PI}" />
     </finger_fixed>
-  </macro>
+  </xacro:macro>
 </robot>

File: turtlebot_arm_description/urdf/arm_hardware.xacro (robot description, xacro)
@@ -1,13 +1,13 @@
 <?xml version="1.0"?>
-<robot>
-  <property name="M_PI" value="3.14159"/>
-  <property name="M_SCALE" value="0.001"/>
-  <property name="F10_HEIGHT" value="0.004"/>
-  <property name="F4_HEIGHT" value="0.0525"/>
-  <property name="F3_HEIGHT" value="0.009"/>
-  <property name="AX12_HEIGHT" value="0.0385"/>
-  <property name="AX12_WIDTH" value="0.038"/>
-  <property name="F2_HEIGHT" value="0.0265"/>
-  <macro name="bioloid_F10_fixed" params="parent name color *origin">
+<robot xmlns:xacro="http://ros.org/wiki/xacro">
+  <xacro:property name="M_PI" value="3.14159"/>
+  <xacro:property name="M_SCALE" value="0.001"/>
+  <xacro:property name="F10_HEIGHT" value="0.004"/>
+  <xacro:property name="F4_HEIGHT" value="0.0525"/>
+  <xacro:property name="F3_HEIGHT" value="0.009"/>
+  <xacro:property name="AX12_HEIGHT" value="0.0385"/>
+  <xacro:property name="AX12_WIDTH" value="0.038"/>
+  <xacro:property name="F2_HEIGHT" value="0.0265"/>
+  <xacro:macro name="bioloid_F10_fixed" params="parent name color *origin">
     <joint name="${name}_joint" type="fixed">
       <insert_block name="origin" />
@@ -37,6 +37,6 @@
       </collision>
     </link>
-  </macro>
-  <macro name="arm_mount" params="parent name color *origin">
+  </xacro:macro>
+  <xacro:macro name="arm_mount" params="parent name color *origin">
     <joint name="${name}_joint" type="fixed">
       <insert_block name="origin" />
@@ -66,6 +66,6 @@
       </collision>
     </link>
-  </macro>
-  <macro name="finger_fixed" params="parent name color *origin">
+  </xacro:macro>
+  <xacro:macro name="finger_fixed" params="parent name color *origin">
     <joint name="${name}_joint" type="fixed">
       <insert_block name="origin" />
@@ -95,6 +95,6 @@
       </collision>
     </link>
-  </macro>
-  <macro name="bioloid_F3_fixed" params="parent name color *origin">
+  </xacro:macro>
+  <xacro:macro name="bioloid_F3_fixed" params="parent name color *origin">
     <joint name="${name}_joint" type="fixed">
       <insert_block name="origin" />
@@ -124,6 +124,6 @@
       </collision>
     </link>
-  </macro>
-  <macro name="dynamixel_AX12_fixed" params="parent name *origin">
+  </xacro:macro>
+  <xacro:macro name="dynamixel_AX12_fixed" params="parent name *origin">
     <joint name="${name}_joint" type="fixed">
       <insert_block name="origin" />
@@ -153,6 +153,6 @@
       </collision>
     </link>
-  </macro>
-  <macro name="bioloid_F3_revolute" params="parent name color llimit ulimit vlimit *origin">
+  </xacro:macro>
+  <xacro:macro name="bioloid_F3_revolute" params="parent name color llimit ulimit vlimit *origin">
     <joint name="${name}_joint" type="revolute">
       <insert_block name="origin" />
@@ -184,6 +184,6 @@
       </collision>
     </link>
-  </macro>
-  <macro name="bioloid_F2_revolute" params="parent name color llimit ulimit vlimit *origin">
+  </xacro:macro>
+  <xacro:macro name="bioloid_F2_revolute" params="parent name color llimit ulimit vlimit *origin">
     <joint name="${name}_joint" type="revolute">
       <insert_block name="origin" />
@@ -215,6 +215,6 @@
       </collision>
     </link>
-  </macro>
-  <macro name="bioloid_F4_revolute" params="parent name color llimit ulimit vlimit *origin">
+  </xacro:macro>
+  <xacro:macro name="bioloid_F4_revolute" params="parent name color llimit ulimit vlimit *origin">
     <joint name="${name}_joint" type="revolute">
       <insert_block name="origin" />
@@ -246,4 +246,4 @@
       </collision>
     </link>
-  </macro>
+  </xacro:macro>
 </robot>

Commit message: Turtlebot arm macro: we can now configure joints velocity limit (same value for all) and lower/upper limits for the first joint (arm_shoulder_pan) to allow accessing to different operational areas, e.g. left handed (as in the turtlebot_arm building tutorial) vs. right handed robot vs. centered arm robot

File: turtlebot_arm_description/urdf/arm.urdf.xacro (robot description, xacro)
@@ -11,5 +11,9 @@
     <!-- Instead, there is a base_link -->
     <link name="base_link"/>
-    <turtlebot_arm parent="base_link" color="white" gripper_color="green">
+    <!-- Turtlebot arm macro: we can configure joints velocity limit and lower/upper limits
+         for the first joint (arm_shoulder_pan) to allow accessing to different operational
+         areas, e.g. left handed vs. right handed robot -->
+    <turtlebot_arm parent="base_link" color="white" gripper_color="green"
+                   joints_vlimit="1.571" pan_llimit="-2.617" pan_ulimit="2.617">
       <origin xyz="0 0 0"/>
     </turtlebot_arm>

File: turtlebot_arm_description/urdf/arm.xacro (robot description, xacro)
@@ -11,5 +11,6 @@
     <color rgba="0.22 0.32 0.14 1.0"/>
   </material>
-  <xacro:macro name="turtlebot_arm" params="parent color gripper_color *origin">
+  <xacro:macro name="turtlebot_arm" params="parent color gripper_color *origin
+                                            joints_vlimit pan_llimit pan_ulimit">
     <link name="arm_base_link" />
     <joint name="arm_base_joint" type="fixed">
@@ -33,5 +34,6 @@
       <origin xyz="0 0 0" rpy="${M_PI/2} 0 ${M_PI/2}"/>
     </dynamixel_AX12_fixed>
-    <bioloid_F3_revolute parent="arm_shoulder_pan_servo_link" name="arm_shoulder_pan" color="${color}" vlimit="0.785" llimit="-2.617" ulimit="2.617">
+    <bioloid_F3_revolute parent="arm_shoulder_pan_servo_link" name="arm_shoulder_pan" color="${color}"
+                         vlimit="${joints_vlimit}" llimit="${pan_llimit}" ulimit="${pan_ulimit}">
       <origin xyz="0 ${AX12_WIDTH/2} 0" rpy="${-M_PI/2} ${M_PI/2} ${M_PI}" />
     </bioloid_F3_revolute>
@@ -40,5 +42,6 @@
       <origin xyz="0 0 ${-AX12_HEIGHT-F10_HEIGHT+0.001}" rpy="0 ${M_PI} 0" />
     </dynamixel_AX12_fixed>
-    <bioloid_F4_revolute parent="arm_shoulder_lift_servo_link" name="arm_shoulder_lift" color="${color}" vlimit="1.571" llimit="-2.617" ulimit="2.617">
+    <bioloid_F4_revolute parent="arm_shoulder_lift_servo_link" name="arm_shoulder_lift" color="${color}"
+                         vlimit="${joints_vlimit}" llimit="-2.617" ulimit="2.617">
       <origin xyz="0 0 0" rpy="0 0 0" />
     </bioloid_F4_revolute>
@@ -59,5 +62,6 @@
       <origin xyz="0 0 ${-AX12_HEIGHT-F10_HEIGHT+0.001}" rpy="0 ${M_PI} 0"/>
     </dynamixel_AX12_fixed>
-    <bioloid_F4_revolute parent="arm_elbow_flex_servo_link" name="arm_elbow_flex" color="${color}" vlimit="1.571" llimit="-2.617" ulimit="2.617">
+    <bioloid_F4_revolute parent="arm_elbow_flex_servo_link" name="arm_elbow_flex" color="${color}"
+                         vlimit="${joints_vlimit}" llimit="-2.617" ulimit="2.617">
       <origin xyz="0 0 0" rpy="0 0 0" />
     </bioloid_F4_revolute>
@@ -78,5 +82,6 @@
       <origin xyz="0 0 ${-AX12_HEIGHT-F10_HEIGHT+0.001}" rpy="0 ${M_PI} 0"/>
     </dynamixel_AX12_fixed>
-    <bioloid_F2_revolute parent="arm_wrist_flex_servo_link" name="arm_wrist_flex" color="${color}" vlimit="1.571" llimit="-1.745" ulimit="1.745">
+    <bioloid_F2_revolute parent="arm_wrist_flex_servo_link" name="arm_wrist_flex" color="${color}"
+                         vlimit="${joints_vlimit}" llimit="-1.745" ulimit="1.745">
       <origin xyz="0 0 0" rpy="0 0 0" />
     </bioloid_F2_revolute>
